File: hardware/EspCnc.kicad_sch (KiCad schematic)
At the start: 0 parts

Commit message: EspCnc usinado
Signed-off-by: cukier <mauricio@krebs.com.br>
Parts:
- added H1, H2, H3, H4: MountingHole_Pad, MountingHole:MountingHole_3.7mm_Pad, symbol Mechanical:MountingHole_Pad
Connections:
- new net GND: H1.1, H2.1, H3.1, H4.1
- no-connect marks 0 -> 11
Other:
- added sheet limits (limits.kicad_sch)
- added sheet motion (motion.kicad_sch)
- sheet core ports: added BOOT, CHIP_PU, GPIO02, GPIO04, GPIO05, GPIO12, GPIO13, GPIO14, GPIO15, GPIO16, GPIO17, GPIO18, GPIO19, GPIO21, GPIO22, GPIO23, GPIO25, GPIO26, GPIO27, GPIO32, GPIO33, GPIO34, GPIO35, GPIO36, GPIO39, U0_RX, U0_TX; removed none
- sheet usb ports: added EN, IO0, RX, TX; removed none
