File: hardware/EspCnc.kicad_pcb (KiCad board)
At the start: 2 copper layers, 0 parts

Commit message: EspCnc usinado
Signed-off-by: cukier <mauricio@krebs.com.br>
Parts:
- added A1: A4988, Module:Pololu_Breakout-16_15.2x20.3mm, F.Cu at (61.1, 141.3)
- added A2: A4988, Module:Pololu_Breakout-16_15.2x20.3mm, F.Cu at (85.6, 141.3)
- added A3: A4988, Module:Pololu_Breakout-16_15.2x20.3mm, F.Cu at (109.7, 141.3)
- added C1: 470uF, Capacitor_THT:CP_Radial_D13.0mm_P5.00mm, F.Cu at (64.2, 71.7)
- added C10: 100nF, Capacitor_SMD:C_1206_3216Metric, B.Cu at (112.2, 63.5)
- added C11: 100uF, Capacitor_THT:CP_Radial_D5.0mm_P2.50mm, F.Cu at (77.2, 136.2)
- added C12: 100nF, Capacitor_SMD:C_1206_3216Metric, B.Cu at (82.0, 140.0)
- added C13: 100uF, Capacitor_THT:CP_Radial_D5.0mm_P2.50mm, F.Cu at (101.8, 136.2)
- added C14: 100nF, Capacitor_SMD:C_1206_3216Metric, B.Cu at (106.5, 139.8)
- added C15: 100uF, Capacitor_THT:CP_Radial_D5.0mm_P2.50mm, F.Cu at (126.0, 136.5)
- added C16: 100nF, Capacitor_SMD:C_1206_3216Metric, B.Cu at (130.5, 138.5)
- added C17: 100nF, Capacitor_SMD:C_1206_3216Metric, B.Cu at (63.5, 106.5)
- added C18: 100nF, Capacitor_SMD:C_1206_3216Metric, B.Cu at (55.8, 82.5)
- added C19: 100nF, Capacitor_SMD:C_1206_3216Metric, B.Cu at (67.2, 87.0)
- added C2: 100nF, Capacitor_SMD:C_1206_3216Metric, B.Cu at (55.0, 70.8)
- added C20: 100nF, Capacitor_SMD:C_1206_3216Metric, B.Cu at (59.2, 93.8)
- added C21: 100nF, Capacitor_SMD:C_1206_3216Metric, B.Cu at (55.8, 99.5)
- added C3: 1000uF, Capacitor_THT:CP_Radial_D10.0mm_P5.00mm, F.Cu at (74.0, 81.6)
- added C4: 100nF, Capacitor_SMD:C_1206_3216Metric, B.Cu at (69.2, 74.2)
- added C5: 22uF, Capacitor_THT:CP_Radial_D8.0mm_P3.50mm, F.Cu at (91.4, 66.8)
- added C6: 100nF, Capacitor_SMD:C_1206_3216Metric, B.Cu at (95.8, 63.2)
- added C7: 1uF, Capacitor_SMD:C_1206_3216Metric, B.Cu at (101.0, 80.0)
- added C8: 100nF, Capacitor_SMD:C_1206_3216Metric, B.Cu at (99.0, 78.0)
- added C9: 1uF, Capacitor_SMD:C_1206_3216Metric, B.Cu at (112.2, 60.1)
- added D1: US1M, Diode_SMD:D_SMA, B.Cu at (55.0, 64.5)
- added D10: BZx558v2, Diode_SMD:D_MELF_Handsoldering, B.Cu at (63.5, 101.2)
- added D2: PWR, LED_THT:LED_D3.0mm, F.Cu at (73.7, 110.0)
- added D3: B340, Diode_SMD:D_SMC, B.Cu at (89.0, 74.0)
- added D4: US1M, Diode_SMD:D_SMA, B.Cu at (89.0, 63.2)
- added D5: SS34, Diode_SMD:D_SMA_Handsoldering, B.Cu at (65.5, 120.2)
- added D6: SPINDLE, LED_THT:LED_D3.0mm, F.Cu at (59.8, 107.5)
- added D7: BZx558v2, Diode_SMD:D_MELF_Handsoldering, B.Cu at (66.0, 82.8)
- added D8: BZx558v2, Diode_SMD:D_MELF_Handsoldering, B.Cu at (69.2, 90.5)
- added D9: BZx558v2, Diode_SMD:D_MELF_Handsoldering, B.Cu at (69.2, 94.8)
- added H1: MountingHole_Pad, MountingHole:MountingHole_3.7mm_Pad, F.Cu at (55.0, 55.0)
- added H2: MountingHole_Pad, MountingHole:MountingHole_3.7mm_Pad, F.Cu at (133.5, 55.0)
- added H3: MountingHole_Pad, MountingHole:MountingHole_3.7mm_Pad, F.Cu at (55.0, 145.0)
- added H4: MountingHole_Pad, MountingHole:MountingHole_3.7mm_Pad, F.Cu at (133.5, 145.0)
- added J1: PWR, Connector_BarrelJack:BarrelJack_Horizontal, F.Cu at (64.2, 64.0)
- added J10: LIMITS, Connector_PinHeader_2.54mm:PinHeader_2x04_P2.54mm_Vertical, F.Cu at (53.2, 87.2)
- added J2: ESP_32, Connector_PinSocket_2.54mm:PinSocket_2x09_P2.54mm_Vertical, F.Cu at (111.0, 111.9)
- added J3: ESP_32, Connector_PinSocket_2.54mm:PinSocket_2x09_P2.54mm_Vertical, F.Cu at (111.0, 84.0)
- added J4: USB_E, Connector_PinSocket_2.54mm:PinSocket_1x09_P2.54mm_Vertical, F.Cu at (103.5, 71.7)
- added J5: USB_D, Connector_PinSocket_2.54mm:PinSocket_1x09_P2.54mm_Vertical, F.Cu at (103.5, 56.5)
- added J6: STEPPER, Connector_PinHeader_2.54mm:PinHeader_1x04_P2.54mm_Vertical, F.Cu at (66.2, 147.8)
- added J7: STEPPER, Connector_PinHeader_2.54mm:PinHeader_1x04_P2.54mm_Vertical, F.Cu at (90.7, 147.8)
- added J8: STEPPER, Connector_PinHeader_2.54mm:PinHeader_1x04_P2.54mm_Vertical, F.Cu at (114.7, 147.8)
- added J9: SPINDLE, TerminalBlock_Phoenix:TerminalBlock_Phoenix_MKDS-1,5-2-5.08_1x02_P5.08mm_Horizontal, F.Cu at (55.3, 117.7)
- added L1: 100uH, Inductor_SMD:L_Changjiang_FXL0840, B.Cu at (77.5, 74.0)
- added Q1: PN2222A, Package_TO_SOT_THT:TO-92L_Inline_Wide, F.Cu at (115.5, 93.7)
- added Q2: PN2222A, Package_TO_SOT_THT:TO-92L_Inline_Wide, F.Cu at (126.7, 98.8)
- added Q3: IRF540N, Package_TO_SOT_THT:TO-220-3_Vertical, F.Cu at (66.0, 110.8)
- added Q4: BC337, Package_TO_SOT_THT:TO-92_Inline_Wide, F.Cu at (88.6, 89.0)
- added Q5: BC337, Package_TO_SOT_THT:TO-92_Inline_Wide, F.Cu at (82.9, 89.2)
- added Q6: BC337, Package_TO_SOT_THT:TO-92_Inline_Wide, F.Cu at (84.9, 96.7)
- added Q7: BC337, Package_TO_SOT_THT:TO-92_Inline_Wide, F.Cu at (76.2, 103.8)
- added R1: 10k, Resistor_SMD:R_1206_3216Metric, B.Cu at (80.8, 110.0)
- added R10: 10k, Resistor_SMD:R_1206_3216Metric, B.Cu at (103.5, 124.0)
- added R11: 10k, Resistor_SMD:R_1206_3216Metric, B.Cu at (101.0, 124.0)
- added R12: 10k, Resistor_SMD:R_1206_3216Metric, B.Cu at (98.2, 124.0)
- added R13: 10k, Resistor_SMD:R_1206_3216Metric, B.Cu at (95.8, 124.0)
- added R14: 10k, Resistor_SMD:R_1206_3216Metric, B.Cu at (127.8, 123.8)
- added R15: 10k, Resistor_SMD:R_1206_3216Metric, B.Cu at (125.0, 123.8)
- added R16: 10k, Resistor_SMD:R_1206_3216Metric, B.Cu at (122.2, 123.8)
- added R17: 10k, Resistor_SMD:R_1206_3216Metric, B.Cu at (119.5, 123.8)
- added R18: 10R, Resistor_SMD:R_1206_3216Metric, B.Cu at (69.0, 106.5)
- added R19: 10k, Resistor_SMD:R_1206_3216Metric, B.Cu at (66.2, 106.5)
- added R2: 10k, Resistor_SMD:R_1206_3216Metric, B.Cu at (121.2, 97.8)
- added R20: 4k7, Resistor_SMD:R_1206_3216Metric, B.Cu at (56.0, 106.5)
- added R21: 10k, Resistor_SMD:R_1206_3216Metric, B.Cu at (58.5, 82.5)
- added R22: 10k, Resistor_SMD:R_1206_3216Metric, B.Cu at (82.2, 86.5)
- added R23: 10k, Resistor_SMD:R_1206_3216Metric, B.Cu at (94.8, 88.5)
- added R24: 10k, Resistor_SMD:R_1206_3216Metric, B.Cu at (61.8, 88.5)
- added R25: 10k, Resistor_SMD:R_1206_3216Metric, B.Cu at (77.8, 90.5)
- added R26: 10k, Resistor_SMD:R_1206_3216Metric, B.Cu at (94.8, 91.2)
- added R27: 10k, Resistor_SMD:R_1206_3216Metric, B.Cu at (62.0, 93.8)
- added R28: 10k, Resistor_SMD:R_1206_3216Metric, B.Cu at (77.8, 94.8)
- added R29: 10k, Resistor_SMD:R_1206_3216Metric, B.Cu at (94.8, 94.0)
- added R3: 10k, Resistor_SMD:R_1206_3216Metric, B.Cu at (112.1, 90.0)
- added R30: 10k, Resistor_SMD:R_1206_3216Metric, B.Cu at (52.8, 99.5)
- added R31: 10k, Resistor_SMD:R_1206_3216Metric, B.Cu at (72.0, 101.2)
- added R32: 10k, Resistor_SMD:R_1206_3216Metric, B.Cu at (79.8, 99.8)
- added R33: 10k, Resistor_SMD:R_1206_3216Metric, B.Cu at (80.6, 103.8)
- added R4: 10k, Resistor_SMD:R_1206_3216Metric, B.Cu at (121.2, 94.8)
- added R5: 10k, Resistor_SMD:R_1206_3216Metric, B.Cu at (130.1, 89.8)
- added R6: 10k, Resistor_SMD:R_1206_3216Metric, B.Cu at (78.8, 124.0)
- added R7: 10k, Resistor_SMD:R_1206_3216Metric, B.Cu at (76.2, 124.0)
- added R8: 10k, Resistor_SMD:R_1206_3216Metric, B.Cu at (73.8, 124.0)
- added R9: 10k, Resistor_SMD:R_1206_3216Metric, B.Cu at (71.2, 124.0)
- added SW1: MS, Button_Switch_THT:SW_DIP_SPSTx03_Slide_6.7x9.18mm_W7.62mm_P2.54mm_LowProfile, F.Cu at (63.7, 132.5)
- added SW2: MS, Button_Switch_THT:SW_DIP_SPSTx03_Slide_6.7x9.18mm_W7.62mm_P2.54mm_LowProfile, F.Cu at (88.2, 132.5)
- added SW3: MS, Button_Switch_THT:SW_DIP_SPSTx03_Slide_6.7x9.18mm_W7.62mm_P2.54mm_LowProfile, F.Cu at (112.2, 132.5)
- added U1: LM2576HVS-5, Package_TO_SOT_SMD:TO-263-5_TabPin3, B.Cu at (77.5, 57.2)
- added U2: AMS1117-3.3, Package_TO_SOT_SMD:SOT-223-3_TabPin2, B.Cu at (90.0, 56.0)
Routing:
- net +12V: track 0.00 -> 384.2 mm, vias 0 -> 12
- net +3V3: track 0.00 -> 365.5 mm, vias 0 -> 12
- net /SPINDLE: track 0.00 -> 100.0 mm
- net +5V: track 0.00 -> 96.5 mm, vias 0 -> 2
- net /X_STEP: track 0.00 -> 94.6 mm, vias 0 -> 14
- net /STEP_ENABLE: track 0.00 -> 86.0 mm, vias 0 -> 4
- net /X_LIMIT: track 0.00 -> 78.4 mm, vias 0 -> 2
- net /X_DIR: track 0.00 -> 71.9 mm, vias 0 -> 10
- net /Y_LIMIT: track 0.00 -> 63.7 mm, vias 0 -> 2
- net GND: track 0.00 -> 63.7 mm, vias 0 -> 21
- net /Z_STEP: track 0.00 -> 59.3 mm, vias 0 -> 4
- net /Y_DIR: track 0.00 -> 51.6 mm, vias 0 -> 2
- net /usb/DTR: track 0.00 -> 50.9 mm
- net /PROBE: track 0.00 -> 49.2 mm, vias 0 -> 2
- net /Y_STEP: track 0.00 -> 48.9 mm, vias 0 -> 4
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- added copper zone on B.Cu, net GND
Other:
- board outline added: 88.5 x 100 mm
