File: hardware/alim.kicad_sch (KiCad schematic)
At the start: 13 parts, among them J1 PWR, U1 LM2576HVS-5, U2 AMS1117-3.3

Commit message: EspCnc usinado
Signed-off-by: cukier <mauricio@krebs.com.br>
Parts:
- added D2: PWR, LED_THT:LED_D3.0mm, symbol Device:LED
- added R1: 10k, Resistor_SMD:R_1206_3216Metric, symbol Device:R
- renumbered D2 to D3, D3 to D4
Connections:
- net +12V: now also R1.1
- net GND: now also D2.1 (K)
- new net: D2.2 (A), R1.2
