File: hardware/core.kicad_sch (KiCad schematic)
At the start: 3 parts, among them U3 ESP32-WROOM-E

Commit message: EspCnc usinado
Signed-off-by: cukier <mauricio@krebs.com.br>
Parts:
- removed U3: ESP32-WROOM-E, PCM_Espressif:ESP32-WROOM-32E, symbol PCM_Espressif:ESP32-WROOM-E
- added J2, J3: ESP_32, Connector_PinSocket_2.54mm:PinSocket_2x09_P2.54mm_Vertical, symbol Connector_Generic:Conn_02x09_Odd_Even
- C7: renamed from C8; footprint Capacitor_SMD:C_0805_2012Metric -> Capacitor_SMD:C_1206_3216Metric; PartNr GRM21BR71H105KA12L -> (none)
- C8: renamed from C7; footprint Capacitor_SMD:C_0805_2012Metric -> Capacitor_SMD:C_1206_3216Metric; PartNr GCM21BR72A104KA37L -> (none)
Connections:
- net +3V3: now also J3.1 (Pin_1)
- net BOOT: now also J3.16 (Pin_16)
- net CHIP_PU: now also J3.4 (Pin_4)
- net GND: now also J3.2 (Pin_2), J3.7 (Pin_7)
- net GPIO02: now also J3.17 (Pin_17)
- net GPIO04: now also J3.15 (Pin_15)
- net GPIO05: now also J3.18 (Pin_18)
- net GPIO12: now also J2.11 (Pin_11)
- net GPIO13: now also J2.12 (Pin_12)
- net GPIO14: now also J2.10 (Pin_10)
- net GPIO15: now also J3.12 (Pin_12)
- net GPIO16: now also J3.14 (Pin_14)
- net GPIO17: now also J3.13 (Pin_13)
- net GPIO18: now also J3.11 (Pin_11)
- net GPIO19: now also J3.10 (Pin_10)
- net GPIO21: now also J3.9 (Pin_9)
- net GPIO22: now also J3.8 (Pin_8)
- net GPIO23: now also J3.6 (Pin_6)
- net GPIO25: now also J2.7 (Pin_7)
- net GPIO26: now also J2.8 (Pin_8)
- net GPIO27: now also J2.9 (Pin_9)
- net GPIO32: now also J2.5 (Pin_5)
- net GPIO33: now also J2.6 (Pin_6)
- net GPIO34: now also J2.3 (Pin_3)
- net GPIO35: now also J2.4 (Pin_4)
- net GPIO36: now also J2.1 (Pin_1)
- net GPIO39: now also J2.2 (Pin_2)
- net U0_RX: now also J3.5 (Pin_5)
- net U0_TX: now also J3.3 (Pin_3)
- no-connect marks 0 -> 6
