File: hardware/usb.kicad_sch (KiCad schematic)
At the start: 14 parts, among them J2 USB-B1HSXX, Q1 MMDT2222A, U4 USBLC6-2SC6, U5 CH340X

Commit message: EspCnc usinado
Signed-off-by: cukier <mauricio@krebs.com.br>
Parts:
- removed C11: 10uF, Capacitor_SMD:C_0805_2012Metric, symbol Device:C
- removed C12: 100nF, Capacitor_SMD:C_0805_2012Metric, symbol Device:C
- removed D4: B340, Diode_SMD:D_SMC, symbol Diode:B340
- removed FB1: 120Ω@100MHz, Inductor_SMD:L_0805_2012Metric, symbol Device:FerriteBead
- removed J2: USB-B1HSXX, Connector_USB:USB_B_OST_USB-B1HSxx_Horizontal, symbol Connector:USB_B
- removed Q1: MMDT2222A, Package_TO_SOT_SMD:SOT-363_SC-70-6, symbol Transistor_BJT:MMDT2222A
- removed R1: 12k, Resistor_SMD:R_0805_2012Metric, symbol Device:R
- removed U4: USBLC6-2SC6, Package_TO_SOT_SMD:SOT-23-6, symbol Power_Protection:USBLC6-2SC6
- removed U5: CH340X, Package_SO:MSOP-10_3x3mm_P0.5mm, symbol Interface_USB:CH340X
- added J4: USB_E, Connector_PinSocket_2.54mm:PinSocket_1x09_P2.54mm_Vertical, symbol Connector_Generic:Conn_01x09
- added J5: USB_D, Connector_PinSocket_2.54mm:PinSocket_1x09_P2.54mm_Vertical, symbol Connector_Generic:Conn_01x09
- added Q1, Q2: PN2222A, Package_TO_SOT_THT:TO-92L_Inline_Wide, symbol Transistor_BJT:PN2222A
- added R5: 10k, Resistor_SMD:R_1206_3216Metric, symbol Device:R
- C10: footprint Capacitor_SMD:C_0805_2012Metric -> Capacitor_SMD:C_1206_3216Metric; PartNr GCM21BR72A104KA37L -> (none)
- C9: footprint Capacitor_SMD:C_0805_2012Metric -> Capacitor_SMD:C_1206_3216Metric; PartNr GRM21BR71H105KA12L -> (none)
- R2, R3, R4: value 12k -> 10k; footprint Resistor_SMD:R_0805_2012Metric -> Resistor_SMD:R_1206_3216Metric; PartNr RC0805FR-0712KL -> (none)
Connections:
- net +3V3: now also C10.1, C9.1, J5.5 (Pin_5), R5.2; no longer R4.1
- net +5V: now also J5.4 (Pin_4)
- net GND: now also J4.7 (Pin_7), J5.1 (Pin_1)
- net RX: now also J4.5 (Pin_5)
- net TX: now also J4.1 (Pin_1)
- net VCC: now also J4.4 (Pin_4); no longer C10.1, C9.1
- net at R2.1: now also Q1.2 (B)
- net DTR: now reaches R2.2
- net DTR: now also J4.2 (Pin_2), Q2.1 (E)
- net BOOT renamed RTS
- net RTS: now also J4.3 (Pin_3), Q1.1 (E)
- net CHIP_PU renamed EN
- net EN: now also Q1.3 (C)
- new net: Q2.2 (B), R4.1
- new net CTS: J5.6 (Pin_6)
- new net DCD: J4.9 (Pin_9)
- new net IO0: Q2.3 (C), R5.1
- new net PWREN: J5.8 (Pin_8)
- new net RI: J4.6 (Pin_6)
- new net RSD: J4.8 (Pin_8)
- new net RXL: J5.3 (Pin_3)
- new net SLEEP: J5.7 (Pin_7)
- new net TEN: J5.9 (Pin_9)
- new net TXL: J5.2 (Pin_2)
- no-connect marks 1 -> 9
