File: hardware/Head/Head.kicad_pcb (KiCad board)
At the start: 2 copper layers, 77 x 70 mm, 35 parts, among them J1 HEAD, J2 Conn_01x08, J3 PWR, J4 ESP_32, J5 ESP_32, J6 USB_E, J7 USB_D, Q1 PN2222A, Q2 PN2222A, U1 LM2576HVS-5, U2 AMS1117-3.3

Commit message: head
Signed-off-by: cukier <mauricio@krebs.com.br>
Parts:
- moved Q2 32.1 mm to (66.0, 30.3), turned to 180 degrees
- moved R4 31.8 mm to (65.3, 26.8), turned to 0 degrees
- moved R2 30.2 mm to (67.8, 34.3), turned to 180 degrees
- moved Q1 28.2 mm to (69.7, 31.2), turned to 0 degrees
- moved C9 5.75 mm to (63.0, 44.0)
- moved C8 3.09 mm to (81.0, 28.0), turned to 0 degrees
- moved C7 2.02 mm to (81.0, 30.8), turned to 0 degrees
- moved R5 1.80 mm to (86.0, 55.5), turned to -90 degrees
Routing:
- net /BOOT: track 9.77 -> 68.1 mm, vias 0 -> 2
- net /usb/DTR: track 57.6 -> 11.3 mm, vias 4 -> 0
- net /CH_PU: track 8.61 -> 51.8 mm, vias 0 -> 6
- net GND: track 21.5 -> 63.2 mm, vias 8 -> 14
- net /Y_STEP: track 68.8 -> 42.5 mm, vias 4 -> 0
- net /X_DIR: track 48.4 -> 71.7 mm, vias 0 -> 2
- net /usb/RTS: track 49.8 -> 27.0 mm, vias 4 -> 0
- net /Y_LIMIT: track 53.9 -> 37.4 mm, vias 4 -> 0
- net /U0TX: track 28.9 -> 15.2 mm
- net /STEP_EN: track 82.3 -> 72.0 mm, vias 4 -> 2
- net /Z_LIMIT: track 35.3 -> 45.1 mm, vias 2 -> 0
- net +12V: track 83.3 -> 89.6 mm, vias 2 -> 4
- net +5V: track 82.5 -> 88.0 mm
- net /Z_DIR: track 44.6 -> 48.6 mm, vias 4 -> 0
- net /SPINDLE: track 17.2 -> 20.2 mm, vias 0 -> 2
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