File: hardware/Body/input_nf.kicad_sch (KiCad schematic)
At the start: 7 parts, among them Q7 BC337

Commit message: body
Signed-off-by: cukier <mauricio@krebs.com.br>
Parts:
- removed C21: 100nF, Capacitor_SMD:C_1206_3216Metric, symbol Device:C
- removed D10: BZx558v2, Diode_SMD:D_MELF_Handsoldering, symbol Device:D_Zener
- removed Q7: BC337, Package_TO_SOT_THT:TO-92_Inline_Wide, symbol Transistor_BJT:BC337
- removed R30, R31, R32, R33: 10k, Resistor_SMD:R_1206_3216Metric, symbol Device:R
- added C1: 100nF, Capacitor_SMD:C_1206_3216Metric_Pad1.33x1.80mm_HandSolder, symbol Device:C
- added D1: BZx558v2, Diode_SMD:D_MELF_Handsoldering, symbol Device:D_Zener
- added Q1: BC337, Package_TO_SOT_THT:TO-92_Inline_Wide, symbol Transistor_BJT:BC337
- added R1, R2, R3: 10k, Resistor_SMD:R_1206_3216Metric_Pad1.30x1.75mm_HandSolder, symbol Device:R
Connections:
- net +3V3: now also R3.1
- net GND: now also C1.2, Q1.3 (E), R1.2
- new net: Q1.2 (B), R2.1
- new net: D1.2 (A), R2.2
- new net ALARM: Q1.1 (C), R3.2
- new net LIMIT: C1.1, D1.1 (K), R1.1
