File: hardware/Body/limits.kicad_sch (KiCad schematic)
At the start: 1 part, among them J10 LIMITS

Commit message: body
Signed-off-by: cukier <mauricio@krebs.com.br>
Parts:
- renumbered J10 to J3
Changed lines of the file:
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@@
 		(dnp no)
 		(fields_autoplaced yes)
-		(property "Reference" "J10"
+		(property "Reference" "J3"
 			(at 123.19 82.55 0)
 			(effects
@@
 			(project ""
 				(path "/6f9c8b4e-1c2d-4e3a-9f5a-2b7d0a1c3e4f/8d814227-2890-479d-bd4a-8f227dd79c54"
-					(reference "J10")
+					(reference "J?")
+					(unit 1)
+				)
+			)
+			(project ""
+				(path "/9e3a63c4-e579-41b0-bbee-849c98c6e950/0f8c8205-1814-4895-9f03-c322dd43f987"
+					(reference "J3")
 					(unit 1)
 				)
@@
 		(dnp no)
 		(fields_autoplaced yes)
-		(property "Reference" "#PWR081"
+		(property "Reference" "#PWR04"
 			(at 113.03 90.17 0)
 			(effects
@@
 			(project ""
 				(path "/6f9c8b4e-1c2d-4e3a-9f5a-2b7d0a1c3e4f/8d814227-2890-479d-bd4a-8f227dd79c54"
-					(reference "#PWR081")
+					(reference "#PWR?")
+					(unit 1)
+				)
+			)
+			(project ""
+				(path "/9e3a63c4-e579-41b0-bbee-849c98c6e950/0f8c8205-1814-4895-9f03-c322dd43f987"
+					(reference "#PWR04")
 					(unit 1)
 				)
@@
 		(dnp no)
 		(fields_autoplaced yes)
-		(property "Reference" "#PWR082"
+		(property "Reference" "#PWR05"
 			(at 113.03 104.14 0)
 			(effects
@@
 			(project ""
 				(path "/6f9c8b4e-1c2d-4e3a-9f5a-2b7d0a1c3e4f/8d814227-2890-479d-bd4a-8f227dd79c54"
-					(reference "#PWR082")
+					(reference "#PWR?")
+					(unit 1)
+				)
+			)
+			(project ""
+				(path "/9e3a63c4-e579-41b0-bbee-849c98c6e950/0f8c8205-1814-4895-9f03-c322dd43f987"
+					(reference "#PWR05")
 					(unit 1)
 				)
@@
 				)
 			)
+			(project ""
+				(path "/0f8c8205-1814-4895-9f03-c322dd43f987"
+					(page "#")
+				)
+			)
+			(project "Body"
+				(path "/9e3a63c4-e579-41b0-bbee-849c98c6e950/0f8c8205-1814-4895-9f03-c322dd43f987"
+					(page "6")
+				)
+			)
 		)
 	)
@@
 				)
 			)
+			(project ""
+				(path "/0f8c8205-1814-4895-9f03-c322dd43f987"
+					(page "#")
+				)
+			)
+			(project "Body"
+				(path "/9e3a63c4-e579-41b0-bbee-849c98c6e950/0f8c8205-1814-4895-9f03-c322dd43f987"
+					(page "3")
+				)
+			)
 		)
 	)
@@
 				)
 			)
+			(project ""
+				(path "/0f8c8205-1814-4895-9f03-c322dd43f987"
+					(page "#")
+				)
+			)
+			(project "Body"
+				(path "/9e3a63c4-e579-41b0-bbee-849c98c6e950/0f8c8205-1814-4895-9f03-c322dd43f987"
+					(page "4")
+				)
+			)
 		)
 	)
@@
 				)
 			)
+			(project ""
+				(path "/0f8c8205-1814-4895-9f03-c322dd43f987"
+					(page "#")
+				)
+			)
+			(project "Body"
+				(path "/9e3a63c4-e579-41b0-bbee-849c98c6e950/0f8c8205-1814-4895-9f03-c322dd43f987"
+					(page "5")
+				)
+			)
