File: hardware/Body/spindle.kicad_sch (KiCad schematic)
At the start: 8 parts, among them J9 SPINDLE, Q3 IRF540N

Commit message: body
Signed-off-by: cukier <mauricio@krebs.com.br>
Parts:
- C11: renamed from C17; footprint Capacitor_SMD:C_1206_3216Metric -> Capacitor_SMD:C_1206_3216Metric_Pad1.33x1.80mm_HandSolder
- R26: renamed from R18; footprint Resistor_SMD:R_1206_3216Metric -> Resistor_SMD:R_1206_3216Metric_Pad1.30x1.75mm_HandSolder
- R27: renamed from R19; footprint Resistor_SMD:R_1206_3216Metric -> Resistor_SMD:R_1206_3216Metric_Pad1.30x1.75mm_HandSolder
- R28: renamed from R20; footprint Resistor_SMD:R_1206_3216Metric -> Resistor_SMD:R_1206_3216Metric_Pad1.30x1.75mm_HandSolder
- renumbered J9 to J7, Q3 to Q5
Changed lines of the file:
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@@
 		(dnp no)
 		(fields_autoplaced yes)
-		(property "Reference" "C17"
+		(property "Reference" "C11"
 			(at 171.45 110.4899 0)
 			(effects
@@
 			)
 		)
-		(property "Footprint" "Capacitor_SMD:C_1206_3216Metric"
+		(property "Footprint" "Capacitor_SMD:C_1206_3216Metric_Pad1.33x1.80mm_HandSolder"
 			(at 168.6052 115.57 0)
 			(effects
@@
 			(project "EspCnc"
 				(path "/6f9c8b4e-1c2d-4e3a-9f5a-2b7d0a1c3e4f/82a9eb6b-8101-41b4-a818-d61f117508ec/21fb5a4d-b05a-4fb9-a69b-49a9cdd3184c"
-					(reference "C17")
+					(reference "C?")
+					(unit 1)
+				)
+			)
+			(project "EspCnc"
+				(path "/9e3a63c4-e579-41b0-bbee-849c98c6e950/34ae5d1e-c71f-41e9-8c57-d789a35afc13/21fb5a4d-b05a-4fb9-a69b-49a9cdd3184c"
+					(reference "C11")
 					(unit 1)
 				)
@@
 		(dnp no)
 		(fields_autoplaced yes)
-		(property "Reference" "#PWR076"
+		(property "Reference" "#PWR059"
 			(at 142.24 128.27 0)
 			(effects
@@
 			(project "EspCnc"
 				(path "/6f9c8b4e-1c2d-4e3a-9f5a-2b7d0a1c3e4f/82a9eb6b-8101-41b4-a818-d61f117508ec/21fb5a4d-b05a-4fb9-a69b-49a9cdd3184c"
-					(reference "#PWR076")
+					(reference "#PWR?")
+					(unit 1)
+				)
+			)
+			(project "EspCnc"
+				(path "/9e3a63c4-e579-41b0-bbee-849c98c6e950/34ae5d1e-c71f-41e9-8c57-d789a35afc13/21fb5a4d-b05a-4fb9-a69b-49a9cdd3184c"
+					(reference "#PWR059")
 					(unit 1)
 				)
@@
 		(dnp no)
 		(fields_autoplaced yes)
-		(property "Reference" "R18"
+		(property "Reference" "R26"
 			(at 135.89 104.14 90)
 			(effects
@@
 			)
 		)
-		(property "Footprint" "Resistor_SMD:R_1206_3216Metric"
+		(property "Footprint" "Resistor_SMD:R_1206_3216Metric_Pad1.30x1.75mm_HandSolder"
 			(at 135.89 108.712 90)
 			(effects
@@
 			(project "EspCnc"
 				(path "/6f9c8b4e-1c2d-4e3a-9f5a-2b7d0a1c3e4f/82a9eb6b-8101-41b4-a818-d61f117508ec/21fb5a4d-b05a-4fb9-a69b-49a9cdd3184c"
-					(reference "R18")
+					(reference "R?")
+					(unit 1)
+				)
+			)
+			(project "EspCnc"
+				(path "/9e3a63c4-e579-41b0-bbee-849c98c6e950/34ae5d1e-c71f-41e9-8c57-d789a35afc13/21fb5a4d-b05a-4fb9-a69b-49a9cdd3184c"
+					(reference "R26")
 					(unit 1)
 				)
@@
 		(dnp no)
 		(fields_autoplaced yes)
-		(property "Reference" "R19"
+		(property "Reference" "R27"
 			(at 144.78 115.5699 0)
 			(effects
@@
 			)
 		)
-		(property "Footprint" "Resistor_SMD:R_1206_3216Metric"
+		(property "Footprint" "Resistor_SMD:R_1206_3216Metric_Pad1.30x1.75mm_HandSolder"
 			(at 140.462 116.84 90)
 			(effects
@@
 			(project "EspCnc"
 				(path "/6f9c8b4e-1c2d-4e3a-9f5a-2b7d0a1c3e4f/82a9eb6b-8101-41b4-a818-d61f117508ec/21fb5a4d-b05a-4fb9-a69b-49a9cdd3184c"
-					(reference "R19")
+					(reference "R?")
+					(unit 1)
+				)
+			)
+			(project "EspCnc"
+				(path "/9e3a63c4-e579-41b0-bbee-849c98c6e950/34ae5d1e-c71f-41e9-8c57-d789a35afc13/21fb5a4d-b05a-4fb9-a69b-49a9cdd3184c"
+					(reference "R27")
 					(unit 1)
 				)
@@
 		(dnp no)
 		(fields_autoplaced yes)
-		(property "Reference" "#PWR080"
+		(property "Reference" "#PWR063"
 			(at 167.64 123.19 0)
 			(effects
@@
 			(project "EspCnc"
 				(path "/6f9c8b4e-1c2d-4e3a-9f5a-2b7d0a1c3e4f/82a9eb6b-8101-41b4-a818-d61f117508ec/21fb5a4d-b05a-4fb9-a69b-49a9cdd3184c"
-					(reference "#PWR080")
+					(reference "#PWR?")
+					(unit 1)
+				)
+			)
+			(project "EspCnc"
+				(path "/9e3a63c4-e579-41b0-bbee-849c98c6e950/34ae5d1e-c71f-41e9-8c57-d789a35afc13/21fb5a4d-b05a-4fb9-a69b-49a9cdd3184c"
+					(reference "#PWR063")
 					(unit 1)
 				)
@@
 		(dnp no)
 		(fields_autoplaced yes)
-		(property "Reference" "#PWR077"
+		(property "Reference" "#PWR060"
 			(at 152.4 90.17 0)
 			(effects
@@
 			(project ""
 				(path "/6f9c8b4e-1c2d-4e3a-9f5a-2b7d0a1c3e4f/82a9eb6b-8101-41b4-a818-d61f117508ec/21fb5a4d-b05a-4fb9-a69b-49a9cdd3184c"
-					(reference "#PWR077")
+					(reference "#PWR?")
+					(unit 1)
+				)
+			)
+			(project ""
+				(path "/9e3a63c4-e579-41b0-bbee-849c98c6e950/34ae5d1e-c71f-41e9-8c57-d789a35afc13/21fb5a4d-b05a-4fb9-a69b-49a9cdd3184c"
+					(reference "#PWR060")
 					(unit 1)
 				)
@@
 		(dnp no)
 		(fields_autoplaced yes)
-		(property "Reference" "R20"
+		(property "Reference" "R28"
 			(at 168.91 81.2799 0)
 			(effects
@@
 			)
 		)
-		(property "Footprint" "Resistor_SMD:R_1206_3216Metric"
+		(property "Footprint" "Resistor_SMD:R_1206_3216Metric_Pad1.30x1.75mm_HandSolder"
 			(at 164.592 82.55 90)
 			(effects
@@
 			(project "EspCnc"
 				(path "/6f9c8b4e-1c2d-4e3a-9f5a-2b7d0a1c3e4f/82a9eb6b-8101-41b4-a818-d61f117508ec/21fb5a4d-b05a-4fb9-a69b-49a9cdd3184c"
-					(reference "R20")
+					(reference "R?")
+					(unit 1)
+				)
+			)
+			(project "EspCnc"
+				(path "/9e3a63c4-e579-41b0-bbee-849c98c6e950/34ae5d1e-c71f-41e9-8c57-d789a35afc13/21fb5a4d-b05a-4fb9-a69b-49a9cdd3184c"
+					(reference "R28")
 					(unit 1)
 				)
@@
 		(dnp no)
 		(fields_autoplaced yes)
-		(property "Reference" "J9"
+		(property "Reference" "J7"
 			(at 144.78 82.55 0)
 			(effects
@@
 			(project ""
 				(path "/6f9c8b4e-1c2d-4e3a-9f5a-2b7d0a1c3e4f/82a9eb6b-8101-41b4-a818-d61f117508ec/21fb5a4d-b05a-4fb9-a69b-49a9cdd3184c"
-					(reference "J9")
+					(reference "J?")
+					(unit 1)
+				)
+			)
+			(project ""
+				(path "/9e3a63c4-e579-41b0-bbee-849c98c6e950/34ae5d1e-c71f-41e9-8c57-d789a35afc13/21fb5a4d-b05a-4fb9-a69b-49a9cdd3184c"
+					(reference "J7")
 					(unit 1)
 				)
@@
 			(project ""
 				(path "/6f9c8b4e-1c2d-4e3a-9f5a-2b7d0a1c3e4f/82a9eb6b-8101-41b4-a818-d61f117508ec/21fb5a4d-b05a-4fb9-a69b-49a9cdd3184c"
+					(reference "D?")
+					(unit 1)
+				)
+			)
+			(project ""
+				(path "/9e3a63c4-e579-41b0-bbee-849c98c6e950/34ae5d1e-c71f-41e9-8c57-d789a35afc13/21fb5a4d-b05a-4fb9-a69b-49a9cdd3184c"
 					(reference "D5")
 					(unit 1)
@@
 		(dnp no)
 		(fields_autoplaced yes)
-		(property "Reference" "#PWR079"
+		(property "Reference" "#PWR062"
 			(at 166.37 81.28 0)
 			(effects
@@
 			(project "EspCnc"
 				(path "/6f9c8b4e-1c2d-4e3a-9f5a-2b7d0a1c3e4f/82a9eb6b-8101-41b4-a818-d61f117508ec/21fb5a4d-b05a-4fb9-a69b-49a9cdd3184c"
-					(reference "#PWR079")
+					(reference "#PWR?")
+					(unit 1)
+				)
+			)
+			(project "EspCnc"
+				(path "/9e3a63c4-e579-41b0-bbee-849c98c6e950/34ae5d1e-c71f-41e9-8c57-d789a35afc13/21fb5a4d-b05a-4fb9-a69b-49a9cdd3184c"
+					(reference "#PWR062")
 					(unit 1)
 				)
@@
 		(dnp no)
 		(fields_autoplaced yes)
-		(property "Reference" "#PWR078"
+		(property "Reference" "#PWR061"
 			(at 152.4 124.46 0)
 			(effects
@@
 			(project ""
 				(path "/6f9c8b4e-1c2d-4e3a-9f5a-2b7d0a1c3e4f/82a9eb6b-8101-41b4-a818-d61f117508ec/21fb5a4d-b05a-4fb9-a69b-49a9cdd3184c"
-					(reference "#PWR078")
+					(reference "#PWR?")
+					(unit 1)
+				)
+			)
+			(project ""
+				(path "/9e3a63c4-e579-41b0-bbee-849c98c6e950/34ae5d1e-c71f-41e9-8c57-d789a35afc13/21fb5a4d-b05a-4fb9-a69b-49a9cdd3184c"
+					(reference "#PWR061")
 					(unit 1)
 				)
@@
 		(dnp no)
 		(fields_autoplaced yes)
-		(property "Reference" "Q3"
+		(property "Reference" "Q5"
 			(at 156.21 109.2199 0)
 			(effects
@@
 			(project ""
 				(path "/6f9c8b4e-1c2d-4e3a-9f5a-2b7d0a1c3e4f/82a9eb6b-8101-41b4-a818-d61f117508ec/21fb5a4d-b05a-4fb9-a69b-49a9cdd3184c"
-					(reference "Q3")
+					(reference "Q?")
+					(unit 1)
+				)
+			)
+			(project ""
+				(path "/9e3a63c4-e579-41b0-bbee-849c98c6e950/34ae5d1e-c71f-41e9-8c57-d789a35afc13/21fb5a4d-b05a-4fb9-a69b-49a9cdd3184c"
+					(reference "Q5")
 					(unit 1)
 				)
@@
 			(project ""
 				(path "/6f9c8b4e-1c2d-4e3a-9f5a-2b7d0a1c3e4f/82a9eb6b-8101-41b4-a818-d61f117508ec/21fb5a4d-b05a-4fb9-a69b-49a9cdd3184c"
+					(reference "D?")
+					(unit 1)
+				)
+			)
+			(project ""
+				(path "/9e3a63c4-e579-41b0-bbee-849c98c6e950/34ae5d1e-c71f-41e9-8c57-d789a35afc13/21fb5a4d-b05a-4fb9-a69b-49a9cdd3184c"
 					(reference "D6")
 					(unit 1)
